File: mega485.kicad_pcb (KiCad board)
At the start: 4 copper layers, 101.6 x 53.3 mm, 80 parts, among them J1 Power, J10 Conn_02x01, J11 Conn_02x01, J12 Conn_02x01, J13 Conn_02x01, J14 Conn_02x01, J15 Conn_02x01, J16 Screw_Terminal_01x02, J2 PWM, J3 Analog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

Commit message: Fix incorrect connection between ISO5VA and ISOGNDA (fix associated planes in pcb)
Connections:
- C23 pad 1: ISOGNDA -> ISO5VA
- C25 pad 1: ISOGNDA -> ISO5VA
- C27 pad 1: ISOGNDA -> ISO5VA
- J11 pad 2: ISOGNDA -> ISO5VA
- L4 pad 2: ISOGNDA -> ISO5VA
- R32 pad 1: ISOGNDA -> ISO5VA
- R40 pad 1: ISOGNDA -> ISO5VA
- U9 pad 16: ISOGNDA -> ISO5VA
Routing:
- net ISOGNDA: track 55.9 -> 33.2 mm, vias 11 -> 8
- net ISO5VA: track 0.00 -> 22.6 mm, vias 0 -> 3
- added copper zone on In2.Cu, net ISO5VA
- removed copper zone on In2.Cu, net ISOGNDA
